File: code/claude/kicad-review/references/selftest.kicad_pcb (KiCad board)
At the start: 2 copper layers, 40 x 30 mm, 20 parts, among them J1 HDR, J2 Conn_Coaxial, J3 HDR, U1 MCU_OK, Y1 32.768kHz

Commit message: claude updates
Routing:
- net PAR: track 0.00 -> 20.0 mm
- net PWR: track 0.00 -> 15.0 mm, vias 0 -> 1
Changed lines of the file:
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@@
 		(pad "1" thru_hole circle (at 0 0) (size 1.5 1.5) (drill 0.8) (layers "*.Cu" "*.Mask") (net "GND") (pinfunction "") (pintype "passive"))
 	)
+	(segment (start 0 0) (end 10 0) (width 0.25) (layer "F.Cu") (net "PWR"))
+	(segment (start 10 0) (end 10 5) (width 0.25) (layer "In1.Cu") (net "PWR"))
+	(via (at 10 0) (size 0.6) (drill 0.3) (layers "F.Cu" "B.Cu") (net "PWR"))
+	(segment (start 30 0) (end 40 0) (width 0.25) (layer "F.Cu") (net "PAR"))
+	(segment (start 30 0) (end 40 0) (width 1.0) (layer "F.Cu") (net "PAR"))
 )

Commit message: work on laptop
Routing:
- net +3V3: vias 0 -> 1
Changed lines of the file:
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@@
 	(segment (start 10 0) (end 10 5) (width 0.25) (layer "In1.Cu") (net "PWR"))
 	(via (at 10 0) (size 0.6) (drill 0.3) (layers "F.Cu" "B.Cu") (net "PWR"))
+	(via (at 8.5 8.5) (size 0.45) (drill 0.2) (layers "F.Cu" "B.Cu") (net "+3V3"))
 	(segment (start 30 0) (end 40 0) (width 0.25) (layer "F.Cu") (net "PAR"))
 	(segment (start 30 0) (end 40 0) (width 1.0) (layer "F.Cu") (net "PAR"))
