File: battery.kicad_sch (KiCad schematic)
At the start: 105 parts, among them J10 SOLAR, J9 BAT_PORT, Q10 SI2308, Q11 CSD17581Q3A, Q5 AON7534, Q6 AON7534, Q7 CSD18512Q5B, Q8 CSD18512Q5B, Q9 SI2308, SW3 POWER/RESET, U7 MAX17320G22+, U8 BQ25798

Commit message: change capacitor sizing & update footprints
Parts:
- removed C47: 1uF, Capacitor_SMD:C_0402_1005Metric, symbol Device:C_Small
- added C35: 10uF, Capacitor_SMD:C_1206_3216Metric, symbol Device:C_Small
- SW3: LCSC Part C2681476 -> C202388
Connections:
- net GND: now also C35.2
- net at C71.2, C72.2, C73.2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: now also C35.1

Commit message: assign lcsc part numbers
Parts:
- C35: LCSC Part C14860 -> C33546013
- C57, C59, C60, C63, C65, C71, C73, C74, C82, C84, C85, C86, C87, C88, C92: LCSC Part C49326770 -> C33546013
- C75, C76, C77: LCSC Part C5142571 -> C363542
- R42: LCSC Part C1883546 -> C54530672
- R46, R50: LCSC Part C2902636 -> C54951138
Changed lines of the file:
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@@
 			)
 		)
-		(property "LCSC Part" "C5142571"
+		(property "LCSC Part" "C363542"
 			(at 236.22 106.68 0)
 			(hide yes)
@@
 			)
 		)
-		(property "LCSC Part" "C49326770"
+		(property "LCSC Part" "C33546013"
 			(at 204.47 30.48 0)
 			(hide yes)
@@
 			)
 		)
-		(property "LCSC Part" "C49326770"
+		(property "LCSC Part" "C33546013"
 			(at 140.97 81.28 0)
 			(hide yes)
@@
 			)
 		)
-		(property "LCSC Part" "C49326770"
+		(property "LCSC Part" "C33546013"
 			(at 156.21 81.28 0)
 			(hide yes)
@@
 			)
 		)
-		(property "LCSC Part" "C5142571"
+		(property "LCSC Part" "C363542"
 			(at 236.22 68.58 0)
 			(hide yes)
@@
 			)
 		)
-		(property "LCSC Part" "C49326770"
+		(property "LCSC Part" "C33546013"
 			(at 256.54 90.17 0)
 			(hide yes)
@@
 			)
 		)
-		(property "LCSC Part" "C49326770"
+		(property "LCSC Part" "C33546013"
 			(at 265.43 49.53 0)
 			(hide yes)
@@
 			)
 		)
-		(property "LCSC Part" "C49326770"
+		(property "LCSC Part" "C33546013"
 			(at 261.62 49.53 0)
 			(hide yes)
@@
 			)
 		)
-		(property "LCSC Part" "C5142571"
+		(property "LCSC Part" "C363542"
 			(at 236.22 53.34 0)
 			(hide yes)
@@
 			)
 		)
-		(property "LCSC Part" "C1883546"
+		(property "LCSC Part" "C54530672"
 			(at 63.5 144.78 0)
 			(hide yes)
@@
 			)
 		)
-		(property "LCSC Part" "C49326770"
+		(property "LCSC Part" "C33546013"
 			(at 152.4 81.28 0)
 			(hide yes)
@@
 			)
 		)
-		(property "LCSC Part" "C49326770"
+		(property "LCSC Part" "C33546013"
 			(at 208.28 30.48 0)
 			(hide yes)
@@
 			)
 		)
-		(property "LCSC Part" "C49326770"
+		(property "LCSC Part" "C33546013"
 			(at 275.59 86.36 0)
 			(hide yes)
@@
 			)
 		)
-		(property "LCSC Part" "C49326770"
+		(property "LCSC Part" "C33546013"
 			(at 257.81 49.53 0)
 			(hide yes)
@@
 			)
 		)
-		(property "LCSC Part" "C2902636"
+		(property "LCSC Part" "C54951138"
 			(at 139.7 184.15 0)
 			(hide yes)
@@
 			)
 		)
-		(property "LCSC Part" "C49326770"
+		(property "LCSC Part" "C33546013"
 			(at 198.12 48.26 0)
 			(hide yes)
@@
 			)
 		)
-		(property "LCSC Part" "C2902636"
+		(property "LCSC Part" "C54951138"
 			(at 153.67 158.75 0)
 			(hide yes)
@@
 			)
 		)
-		(property "LCSC Part" "C49326770"
+		(property "LCSC Part" "C33546013"
 			(at 148.59 81.28 0)
 			(hide yes)
@@
 			)
 		)
-		(property "LCSC Part" "C49326770"
+		(property "LCSC Part" "C33546013"
 			(at 254 49.53 0)
 			(hide yes)
@@
 			)
 		)
-		(property "LCSC Part" "C49326770"
+		(property "LCSC Part" "C33546013"
 			(at 144.78 81.28 0)
 			(hide yes)
@@
 			)
 		)
-		(property "LCSC Part" "C49326770"
+		(property "LCSC Part" "C33546013"
 			(at 256.54 86.36 0)
 			(hide yes)
@@
 			)
 		)
-		(property "LCSC Part" "C14860"
+		(property "LCSC Part" "C33546013"
 			(at 196.85 30.48 0)
 			(hide yes)

Commit message: new part numbers for out of stock components
Parts:
- Q11: LCSC Part C2861705 -> C201632
Changed lines of the file:
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@@
 			)
 		)
-		(property "LCSC Part" "C2861705"
+		(property "LCSC Part" "C201632"
 			(at 246.38 95.25 0)
 			(hide yes)

Commit message: backup before switching to kicad-nightly
Parts:
- added C105, C132, C134, C47, C98: 10nF, Capacitor_SMD:C_0402_1005Metric, symbol Device:C_Small
- Q11: value CSD17581Q3A -> CSD17577Q3A
- R51: value 5.24k -> 5.23k
- R52: value 30.31k -> 30.1k
Connections:
- net -BATT: now also C55.1, C56.1, C105.2, C132.2, C47.2, C98.2; no longer C55.2, C56.2
- net GND: now also C134.2
- net at TP3.1, U7.13 (REG3): now also C56.2; no longer C55.1
- net at TH4.1, U7.10 (TH1): now also C47.1
- net at R51.1, R52.2, TH5.1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: now also C134.1
- net at TH1.1, U7.16 (TH2): now also C98.1
- net at U7.17 (REG2): now also C55.2; no longer C56.1
- net at TH3.1, U7.18 (TH3): now also C105.1
- net at TH2.1, U7.19 (TH4): now also C132.1
Other:
- note added: "10nF noise filtering capacitors"
- note removed: "todo: verify sense shunt value"
- moved on the sheet: BT1, BT2, C48, C49, C50, C51, C52, C53, C54, C58, C61, C66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
