File: battery.kicad_sch (KiCad schematic)
At the start: 62 parts, among them J10 SOLAR, Q10 SI2308, Q11 CSD17577Q3A, Q7 CSD18512Q5B, Q8 CSD18512Q5B, Q9 SI2308, SW3 POWER/RESET, U8 BQ25798

Commit message: source slightly larger inductor for higher iSAT
Parts:
- L1: footprint Inductor_SMD:L_Vishay_IFSC-1515AH_4x4x1.8mm -> Inductor_SMD:L_Sunlord_MWSA0503S; JLCPCB Part (none) -> C408408; LCSC Part C5291938 -> (none); MPN (none) -> MWSA0503S-2R2MT
Changed lines of the file:
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@@
 			)
 		)
-		(property "Footprint" "Inductor_SMD:L_Vishay_IFSC-1515AH_4x4x1.8mm"
+		(property "Footprint" "Inductor_SMD:L_Sunlord_MWSA0503S"
 			(at 185.42 83.82 0)
 			(hide yes)
@@
 			)
 		)
-		(property "Description" "Inductor"
+		(property "Description" "2.2uH 29mΩ 7A 7A ±20% SMD,5.4x5.2mm Power Inductors ROHS"
 			(at 185.42 83.82 0)
 			(hide yes)
@@
 			)
 		)
-		(property "LCSC Part" "C5291938"
+		(property "MPN" "MWSA0503S-2R2MT"
 			(at 185.42 83.82 0)
 			(hide yes)
+			(show_name no)
+			(do_not_autoplace no)
+			(effects
+				(font
+					(size 1.27 1.27)
+				)
+			)
+		)
+		(property "LCSC Part" ""
+			(at 185.42 83.82 0)
+			(hide yes)
+			(show_name no)
+			(do_not_autoplace no)
+			(effects
+				(font
+					(size 1.27 1.27)
+				)
+			)
+		)
+		(property "JLCPCB Part" "C408408"
+			(at 185.42 83.82 0)
+			(hide yes)
