File: battery.kicad_sch (KiCad schematic)
At the start: 62 parts, among them J10 SOLAR, Q10 SI2308, Q11 CSD17577Q3A, Q7 CSD18512Q5B, Q8 CSD18512Q5B, Q9 SI2308, SW3 POWER/RESET, U8 BQ25798

Commit message: organize part fields
Parts:
- C134: Dielectric (none) -> X7R; MPN (none) -> TCC0402X7R103M500AT; Manufacturer (none) -> CCTC; Tolerance (none) -> 20%
- C35, C57, C59, C60, C63, C65, C71, C73, C74, C82, C84, C85, C86, C87, C88, C90, C92: Dielectric (none) -> X7R; MPN (none) -> HGC1206R7106K500NSPJ; Manufacturer (none) -> Chinocera; Tolerance (none) -> 10%
- C62, C79: Dielectric (none) -> X7R; MPN (none) -> CS2012X7R225K500NRE; Manufacturer (none) -> Samwha; Tolerance (none) -> 10%
- C64, C72, C80, C89, C91: Capacitor Rating X7R -> (none); Dielectric (none) -> X7R; MPN (none) -> 0402B104J500NT; Manufacturer (none) -> FH (Fenghua); Tolerance (none) -> 5%
- C75, C76, C77: Dielectric (none) -> X7R; MPN (none) -> TCC0402X7R473K500AT; Manufacturer (none) -> CCTC; Tolerance (none) -> 10%
- C78: Dielectric (none) -> X5R; MPN (none) -> HGC0603R5475K350NTHJ; Manufacturer (none) -> Chinocera; Tolerance (none) -> 10%; Voltage Rating 25V -> 35V
- D7: MPN (none) -> SMF24A; Manufacturer (none) -> SUNMATE
- D8: MPN (none) -> YLED0805YG; Manufacturer (none) -> YONGYUTAI
- D9: MPN (none) -> SS36B; Manufacturer (none) -> Baocheng
- J10: MPN (none) -> S2B-PH-SM4-TB(LF)(SN); Manufacturer (none) -> JST
- L1: JLCPCB Part C408408 -> (none); LCSC Part (none) -> C408408; Manufacturer (none) -> Sunlord; Tolerance (none) -> 20%
- Q10, Q9: MPN (none) -> SI2308; Manufacturer (none) -> HXY MOSFET
- Q11: MPN (none) -> CSD17577Q3A; Manufacturer (none) -> Texas Instruments
- Q7, Q8: MPN (none) -> CSD18512Q5B; Manufacturer (none) -> Texas Instruments
- R49, R62: MPN (none) -> FRC0402F2R00TS; Manufacturer (none) -> FOJAN; Power Rating (none) -> 62.5mW; Tolerance (none) -> 1%
- R51: MPN (none) -> RT0603BRD075K23L; Manufacturer (none) -> YAGEO; Power Rating (none) -> 100mW; Tolerance (none) -> 0.1%
- R52: MPN (none) -> TC0325B3012T5F; Manufacturer (none) -> UNI-ROYAL; Power Rating (none) -> 100mW; Tolerance (none) -> 0.1%
- R53, R57, R60, R61: MPN (none) -> RT0402BRD07294RL; Manufacturer (none) -> YAGEO; Power Rating (none) -> 62.5mW; Tolerance (none) -> 0.1%
- R54: MPN (none) -> ARG03BTC2432; Manufacturer (none) -> Viking Tech; Power Rating (none) -> 100mW; Tolerance (none) -> 0.1%
- R55: MPN (none) -> THD03H6812BT; Manufacturer (none) -> FH (Fenghua); Power Rating (none) -> 100mW; Tolerance (none) -> 0.1%
- R56: MPN (none) -> ARG02BTC1003; Manufacturer (none) -> Viking Tech; Power Rating (none) -> 62.5mW; Tolerance (none) -> 0.1%
- R58: MPN (none) -> ARG02BTC8201; Manufacturer (none) -> Viking Tech; Power Rating (none) -> 62.5mW; Tolerance 1% -> 0.1%
- R59, R63: MPN (none) -> FRH0402D1000TS; Manufacturer (none) -> FOJAN; Power Rating (none) -> 62.5mW; Tolerance (none) -> 0.5%
- R64, R65: LCSC Part C54530782 -> C1881139; MPN (none) -> RCS04022R20FKED; Manufacturer (none) -> Vishay; Power Rating (none) -> 200mW; Tolerance (none) -> 1%
- R66: MPN (none) -> TC0225B3001TCC; Manufacturer (none) -> UNI-ROYAL; Power Rating (none) -> 62.5mW; Tolerance (none) -> 0.1%
- SW3: MPN (none) -> SKRKAHE020; Manufacturer (none) -> Alps Alpine
- TH5: value 103AT 10k -> 10k; MPN (none) -> NCU18XH103D60RB; Manufacturer (none) -> Murata; Tolerance (none) -> 0.5%
- U8: MPN (none) -> BQ25798RQMR; Manufacturer (none) -> Texas Instruments

Commit message: add extra PWR_FLAGs
Connections:
- net CHG_VBUS: now reaches C35.1, C71.2, C72.2, C73.2, C74.2, Q8.1 (D), Q9.3 (D), U8.2 (VBUS), U8.3 (VBUS)
Changed lines of the file:
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@@
 	(wire
 		(pts
+			(xy 129.54 48.26) (xy 129.54 50.8)
+		)
+		(stroke
+			(width 0)
+			(type default)
+		)
+	)
+	(wire
+		(pts
 			(xy 198.12 110.49) (xy 203.2 110.49)
 		)
@@
 	(wire
 		(pts
+			(xy 129.54 50.8) (xy 142.24 50.8)
+		)
+		(stroke
+			(width 0)
+			(type default)
+		)
+	)
+	(wire
+		(pts
 			(xy 153.67 52.07) (xy 153.67 50.8)
 		)
@@
 					(unit 1)
 				)
+			)
+		)
+	)
+	(symbol
+		(lib_id "power:VBUS")
+		(at 129.54 48.26 0)
+		(unit 1)
+		(body_style 1)
+		(exclude_from_sim no)
+		(in_bom yes)
+		(on_board yes)
+		(in_pos_files yes)
+		(dnp no)
+		(fields_autoplaced yes)
+		(property "Reference" "#PWR083"
+			(at 129.54 52.07 0)
+			(hide yes)
+			(show_name no)
+			(do_not_autoplace no)
+			(effects
+				(font
+					(size 1.27 1.27)
+				)
+			)
+		)
+		(property "Value" "CHG_VBUS"
+			(at 129.54 43.18 0)
+			(show_name no)
+			(do_not_autoplace no)
+			(effects
+				(font
+					(size 1.27 1.27)
+				)
+			)
+		)
+		(property "Footprint" ""
+			(at 129.54 48.26 0)
+			(hide yes)
+			(show_name no)
+			(do_not_autoplace no)
+			(effects
+				(font
+					(size 1.27 1.27)
+				)
+			)
+		)
+		(property "Datasheet" ""
+			(at 129.54 48.26 0)
+			(hide yes)
+			(show_name no)
+			(do_not_autoplace no)
+			(effects
+				(font
+					(size 1.27 1.27)
+				)
+			)
+		)
+		(property "Description" "Power symbol creates a global label with name \"VBUS\""
+			(at 129.54 48.26 0)
+			(hide yes)
+			(show_name no)
+			(do_not_autoplace no)
+			(effects
+				(font
+					(size 1.27 1.27)
+				)
+			)
+		)
+		(property "MPN" ""
+			(at 129.54 48.26 0)
+			(hide yes)
+			(show_name no)
+			(do_not_autoplace no)
+			(effects
+				(font
+					(size 1.27 1.27)
+				)
+			)
+		)
+		(property "Manufacturer" ""
+			(at 129.54 48.26 0)
+			(hide yes)
+			(show_name no)
+			(do_not_autoplace no)
+			(effects
+				(font
+					(size 1.27 1.27)
+				)
+			)
+		)
+		(property "LCSC Part" ""
+			(at 129.54 48.26 0)
+			(hide yes)
+			(show_name no)
+			(do_not_autoplace no)
+			(effects
+				(font
+					(size 1.27 1.27)
+				)
+			)
+		)
+		(property "Voltage Rating" ""
+			(at 129.54 48.26 0)
+			(hide yes)
+			(show_name no)
+			(do_not_autoplace no)
+			(effects
+				(font
+					(size 1.27 1.27)
+				)
+			)
+		)
+		(property "Tolerance" ""
+			(at 129.54 48.26 0)
+			(hide yes)
+			(show_name no)
+			(do_not_autoplace no)
+			(effects
+				(font
+					(size 1.27 1.27)
+				)
+			)
+		)
+		(pin "1"
+		)
+		(instances
+			(project "parsnip"
+				(path "/c8087976-4958-4446-b419-5a0b61d5634f"
+					(reference "#PWR083")
+					(unit 1)
+				)

Commit message: nearly set to order!
Parts:
- removed J10: SOLAR, Connector_JST:JST_PH_S2B-PH-SM4-TB_1x02-1MP_P2.00mm_Horizontal, symbol Connector:Conn_01x02_Socket
- added J10: SOLAR, Connector_JST:JST_PH_S2B-PH-SM4-TB_1x02-1MP_P2.00mm_Horizontal, symbol Connector_Generic:Conn_01x02
- D7: value SMF24A -> TVS2200DRV; footprint Diode_SMD:D_SOD-123F -> Package_SON:WSON-6-1EP_2x2mm_P0.65mm_EP1x1.6mm; symbol Diode:SMF24A -> Power_Protection:TVS2200DRV; LCSC Part C399294 -> C523793; MPN SMF24A -> TVS2200DRVR; Manufacturer SUNMATE -> Texas Instruments; Note (none) -> VBR 24.6V min (-40..125C), 18mA DC breakdown max: panel col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
Connections:
- net GND: now also D7.1 (GND), D7.3 (GND), D7.7 (GND), J10.2 (Pin_2)
- net SOLAR: now also D7.4 (IN), D7.5 (IN), D7.6 (IN), J10.1 (Pin_1); no longer D7.1 (A1)
Other:
- note added: "Charge Controller with Power Path"
- note added: "R51, R54, R52, R55, all 0.1%"
- note removed: "Capacitors voltage ratings specified, generally >25V - use XR7/C0G"
- note removed: "Charge Controller"
- moved on the sheet: C134, C35, C57, C59, C60, C62, C63, C64, C65, C72, C73, C74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
