File: peripherals.kicad_sch (KiCad schematic)
At the start: 16 parts, among them J14 GPIO_Expander, J15 LED 5V, U17 TCAL9539RTWR, U18 WS2816B, U19 SN74LV1T34DCK, U2 QMC6309, U20 WS2816B

Commit message: organize part fields
Parts:
- C12, C16: Capacitor Rating X7R -> (none); Dielectric (none) -> X5R; MPN (none) -> TCC0603X5R106M350CT; Manufacturer (none) -> CCTC; Tolerance (none) -> 20%; Voltage Rating 16V -> 35V
- C176: Capacitor Rating X7R -> (none); Dielectric (none) -> X7R; MPN (none) -> TCC0402X7R105K250AT; Manufacturer (none) -> CCTC; Tolerance (none) -> 10%
- C178, C179, C180: Dielectric (none) -> X7R; MPN (none) -> TCC0402X7R105K250AT; Manufacturer (none) -> CCTC; Tolerance (none) -> 10%
- C181: Dielectric (none) -> X5R; MPN (none) -> HGC0402R5225K350NTEJ; Manufacturer (none) -> Chinocera; Tolerance (none) -> 10%; Voltage Rating 16V -> 35V
- F6: value 3A hold 5A trip -> 3A hold; MPN (none) -> JSMD1812-300; Manufacturer (none) -> JKSEMI
- J14: MPN (none) -> HX PM2.54-2x8P WT; Manufacturer (none) -> HANXIA
- J15: MPN (none) -> S4B-XH-SM4-TB(LF)(SN); Manufacturer (none) -> JST
- R133: MPN (none) -> FRH0402D1002TS; Manufacturer (none) -> FOJAN; Power Rating (none) -> 62.5mW; Tolerance (none) -> 0.5%
- U17: value TCAL9539RTWR -> TCAL9539RTWRQ1; LCSC Part C22445413 -> C5377958; MPN TCAL9539RTWR -> TCAL9539RTWRQ1; Manufacturer TI(德州仪器) -> Texas Instruments
- U18, U20: Manufacturer worldsemi -> Worldsemi
- U19: MPN (none) -> SN74LV1T34DCKR; Manufacturer (none) -> Texas Instruments
- U2: MPN (none) -> QMC6309; Manufacturer (none) -> QST

Commit message: routing and silkscreen improvements
Parts:
- added C137: 10uF, Capacitor_SMD:C_0603_1608Metric, symbol Device:C_Small
Connections:
- net GND: now also C137.2
- net at F6.2, J15.1 (Pin_1): now also C137.1
Other:
- moved on the sheet: F6
Changed lines of the file:
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@@
 	)
 	(junction
+		(at 252.73 41.91)
+		(diameter 0)
+		(color 0 0 0 0)
+	)
+	(junction
 		(at 132.08 124.46)
 		(diameter 0)
@@
 	)
 	(junction
+		(at 256.54 34.29)
+		(diameter 0)
+		(color 0 0 0 0)
+	)
+	(junction
 		(at 210.82 41.91)
 		(diameter 0)
@@
 	(wire
 		(pts
+			(xy 252.73 34.29) (xy 256.54 34.29)
+		)
+		(stroke
+			(width 0)
+			(type default)
+		)
+	)
+	(wire
+		(pts
 			(xy 177.8 52.07) (xy 177.8 49.53)
 		)
@@
 	(wire
 		(pts
-			(xy 247.65 41.91) (xy 262.89 41.91)
+			(xy 247.65 41.91) (xy 252.73 41.91)
 		)
 		(stroke
@@
 	(wire
 		(pts
-			(xy 262.89 34.29) (xy 260.35 34.29)
+			(xy 262.89 34.29) (xy 256.54 34.29)
 		)
 		(stroke
@@
 	(wire
 		(pts
-			(xy 247.65 31.75) (xy 252.73 31.75)
+			(xy 247.65 31.75) (xy 248.92 31.75)
 		)
 		(stroke
@@
 	(wire
 		(pts
+			(xy 252.73 41.91) (xy 262.89 41.91)
+		)
+		(stroke
+			(width 0)
+			(type default)
+		)
+	)
+	(wire
+		(pts
 			(xy 132.08 128.27) (xy 132.08 124.46)
 		)
@@
 	(wire
 		(pts
+			(xy 252.73 39.37) (xy 252.73 41.91)
+		)
+		(stroke
+			(width 0)
+			(type default)
+		)
+	)
+	(wire
+		(pts
 			(xy 168.91 39.37) (xy 181.61 39.37)
 		)
@@
 	(wire
 		(pts
-			(xy 260.35 34.29) (xy 260.35 31.75)
+			(xy 256.54 34.29) (xy 256.54 31.75)
 		)
 		(stroke
@@
 	(symbol
 		(lib_id "Device:Polyfuse")
-		(at 256.54 31.75 90)
+		(at 252.73 31.75 90)
 		(unit 1)
 		(body_style 1)
@@
 		(dnp no)
 		(property "Reference" "F6"
-			(at 256.54 27.432 90)
+			(at 252.73 27.432 90)
 			(show_name no)
 			(do_not_autoplace no)
@@
 		)
 		(property "Value" "3A hold"
-			(at 257.048 29.464 90)
+			(at 253.238 29.464 90)
 			(show_name no)
 			(do_not_autoplace no)
@@
 		)
 		(property "Footprint" "Fuse:Fuse_1812_4532Metric"
-			(at 261.62 30.48 0)
+			(at 257.81 30.48 0)
 			(hide yes)
 			(show_name no)
@@
 		)
 		(property "Datasheet" "https://datasheet.lcsc.com/datasheet/pdf/82552fc8944c2b3427e6cd651b8d9c76.pdf?productCode=C2972730"
-			(at 256.54 31.75 0)
+			(at 252.73 31.75 0)
 			(hide yes)
 			(show_name no)
@@
 		)
 		(property "Description" "FUSE PTC resettable 3A hold, 5A trip, 6V, 1812"
-			(at 256.54 31.75 0)
+			(at 252.73 31.75 0)
 			(hide yes)
 			(show_name no)
@@
 		)
 		(property "MPN" "JSMD1812-300"
-			(at 261.62 30.48 0)
+			(at 257.81 30.48 0)
 			(hide yes)
 			(show_name no)
@@
 		)
 		(property "Manufacturer" "JKSEMI"
-			(at 261.62 30.48 0)
+			(at 257.81 30.48 0)
 			(hide yes)
 			(show_name no)
@@
 		)
 		(property "LCSC Part" "C2972730"
-			(at 256.54 31.75 0)
+			(at 252.73 31.75 0)
 			(hide yes)
 			(show_name no)
@@
 					(unit 1)
 				)
+			)
+		)
+	)
+	(symbol
+		(lib_id "Device:C_Small")
+		(at 252.73 36.83 0)
+		(unit 1)
+		(body_style 1)
+		(exclude_from_sim no)
+		(in_bom yes)
+		(on_board yes)
+		(in_pos_files yes)
+		(dnp no)
+		(property "Reference" "C137"
+			(at 249.936 40.386 0)
+			(show_name no)
+			(do_not_autoplace no)
+			(effects
+				(font
+					(size 1.27 1.27)
+				)
+				(justify left)
+			)
+		)
+		(property "Value" "10uF"
+			(at 247.396 39.116 0)
+			(hide yes)
+			(show_name no)
+			(do_not_autoplace no)
+			(effects
+				(font
+					(size 1.27 1.27)
+				)
+				(justify left)
+			)
+		)
+		(property "Footprint" "Capacitor_SMD:C_0603_1608Metric"
+			(at 252.73 36.83 0)
+			(hide yes)
+			(show_name no)
+			(do_not_autoplace no)
+			(effects
+				(font
+					(size 1.27 1.27)
+				)
+			)
+		)
+		(property "Datasheet" "https://datasheet.lcsc.com/datasheet/pdf/71a9f8eccc4da164324d4a716182c5e3.pdf?productCode=C22392391"
+			(at 252.73 36.83 0)
+			(hide yes)
+			(show_name no)
+			(do_not_autoplace no)
+			(effects
+				(font
+					(size 1.27 1.27)
+				)
+			)
+		)
+		(property "Description" "CAP MLCC 10uF ±20% 35V X5R 0603"
+			(at 252.73 36.83 0)
+			(hide yes)
+			(show_name no)
+			(do_not_autoplace no)
+			(effects
+				(font
+					(size 1.27 1.27)
+				)
+			)
+		)
+		(property "MPN" "TCC0603X5R106M350CT"
+			(at 252.73 36.83 0)
+			(hide yes)
+			(show_name no)
+			(do_not_autoplace no)
+			(effects
+				(font
+					(size 1.27 1.27)
+				)
+			)
+		)
+		(property "Manufacturer" "CCTC"
+			(at 252.73 36.83 0)
+			(hide yes)
+			(show_name no)
+			(do_not_autoplace no)
+			(effects
+				(font
+					(size 1.27 1.27)
+				)
+			)
+		)
+		(property "LCSC Part" "C22392391"
+			(at 252.73 36.83 0)
+			(hide yes)
+			(show_name no)
+			(do_not_autoplace no)
+			(effects
+				(font
+					(size 1.27 1.27)
+				)
+			)
+		)
+		(property "Voltage Rating" "35V"
+			(at 256.794 39.878 0)
+			(hide yes)
+			(show_name no)
+			(do_not_autoplace no)
+			(effects
+				(font
+					(size 1.27 1.27)
+				)
+			)
+		)
+		(property "Dielectric" "X5R"
+			(at 252.73 36.83 0)
+			(hide yes)
+			(show_name no)
+			(do_not_autoplace no)
+			(effects
+				(font
+					(size 1.27 1.27)
+				)
+			)
+		)
+		(property "Tolerance" "20%"
+			(at 252.73 36.83 0)
+			(hide yes)
+			(show_name no)
+			(do_not_autoplace no)
+			(effects
+				(font
+					(size 1.27 1.27)
+				)
+			)
+		)
+		(pin "1"
+		)
+		(pin "2"
+		)
+		(instances
+			(project "parsnip"
+				(path "/fe9d4a31-2311-442f-997c-52ad8ca5cfe9/8523a718-fda3-4580-a612-9f8de7a7dbdb"
+					(reference "C137")
+					(unit 1)
+				)
