File: peripherals.kicad_sch (KiCad schematic)
At the start: 17 parts, among them J14 GPIO_Expander, J15 LED 5V, U17 TCAL9539RTWRQ1, U18 WS2816B, U19 SN74LV1T34DCK, U2 QMC6309, U20 WS2816B

Commit message: checkpoint: schematic WIP before battery -> charger rename
Connectors and Overview sheets, LSM6DSV16X/TPS22945/charger datasheets,
and in-progress edits across all sheets, committed as-is so the rename
diff stands alone.

Co-Authored-By: Claude Opus 5.5 <noreply@anthropic.com>
Parts:
- added C183, C193: 2.2uF, Capacitor_SMD:C_0402_1005Metric, symbol Device:C_Small
- added U22: LSM6DSV16X, Package_LGA:LGA-14_3x2.5mm_P0.5mm_LayoutBorder3x4y, symbol Sensor_Motion:LSM6DSM
Connections:
- net +3V3: now also C183.1, C193.1, U22.12 (CS), U22.5 (VDDIO), U22.8 (VDD)
- net GND: now also J14.12 (Pin_12), C183.2, C193.2, U22.1 (SDO/SA0), U22.2 (SDX), U22.3 (SCX), U22.6 (GND), U22.7 (GND)
- net I2C_HOST_SCL: now also U22.13 (SCL)
- net I2C_HOST_SDA: now also U22.14 (SDA)
- net P15: now also U22.4 (INT1); no longer J14.12 (Pin_12)
- no-connect marks 0 -> 3
Other:
- title: GPIO Expander / LEDs / Magnetometer -> GPIO Expander, RGB LEDs, Magnetometer
