File: peripherals.kicad_sch (KiCad schematic)
At the start: 20 parts, among them J14 GPIO_Expander, J15 LED 5V, U17 TCAL9539RTWRQ1, U18 WS2816B, U19 SN74LV1T34DCK, U2 QMC6309, U20 WS2816B, U22 LSM6DSV16X

Commit message: schematic reorganization
Parts:
- added U24: TPD2E2U06QDCKRQ1, Package_TO_SOT_SMD:SOT-323_SC-70, symbol Power_Protection:TPD2E2U06DCK
Connections:
- net GND: now also U24.3
- net LED_BDO: now also U24.2
- net LED_DO: now also U24.1
- net P07: no longer names the net of J14.15 (Pin_15)
- net P07: no longer U17.8 (P07)
- new net IO_P07: U17.8 (P07)
- no-connect marks 3 -> 4
Other:
- note added: "IMU"
- moved on the sheet: C12, C137, C16, C178, C179, C180, C183, C193, F6, J14, J15, U18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
