File: peripherals.kicad_sch (KiCad schematic)
At the start: 21 parts, among them J14 GPIO_Expander, J15 LED 5V, U17 TCAL9539RTWRQ1, U18 WS2816B, U19 SN74LV1T34DCK, U2 QMC6309, U20 WS2816B, U22 LSM6DSV16X, U24 TPD2E2U06QDCKRQ1

Commit message: todo fixes
Parts:
- J14: footprint easyeda2kicad:HDR-SMD_16P-P2.54_HXPM2.54-2X8PWT -> footprints:HDR-SMD_16P-P2.54_HXPM2.54-2X8PWT
Changed lines of the file:
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@@
 			)
 		)
-		(property "Footprint" "easyeda2kicad:HDR-SMD_16P-P2.54_HXPM2.54-2X8PWT"
+		(property "Footprint" "footprints:HDR-SMD_16P-P2.54_HXPM2.54-2X8PWT"
 			(at 127 114.3 0)
 			(hide yes)
