File: rails.kicad_sch (KiCad schematic)
At the start: 105 parts, among them Q15 2N7002, U13 LM61460AASQRJRRQ1, U14 LM61460AASQRJRRQ1, U15 TPS259474ARPWR, U16 SN74LVC1G74, Y2 SX1M4.000M10F30TNN

Commit message: change capacitor sizing & update footprints
Parts:
- removed C130, C134: 100nF, Capacitor_SMD:C_0402_1005Metric, symbol Device:C_Small
- removed C132, C138: 1uF, Capacitor_SMD:C_0603_1608Metric, symbol Device:C_Small
- removed C137, C146, C167, C174: 1uF, Capacitor_SMD:C_0402_1005Metric, symbol Device:C_Small
- removed C148, C149, C150, C165, C166, C172, C173, C175: 22uF, Capacitor_SMD:C_1206_3216Metric, symbol Device:C_Small
- removed C151, C154: 10uF, Capacitor_SMD:C_1206_3216Metric, symbol Device:C_Small
- added C177, C188, C189, C190, C191, C192: 10uF, Capacitor_SMD:C_0603_1608Metric, symbol Device:C_Small
- C122, C126, C141, C143: footprint Capacitor_SMD:C_1206_3216Metric -> Capacitor_SMD:C_0603_1608Metric; LCSC Part C49326770 -> C22392391; Voltage Rating 50V -> 35V
- C123, C127: value 1uF -> 10uF; LCSC Part C7432774 -> C22392391; Voltage Rating 50V -> 35V
- C124, C128: value 100nF -> 10uF; footprint Capacitor_SMD:C_0402_1005Metric -> Capacitor_SMD:C_0603_1608Metric; Capacitor Rating X7R -> (none); LCSC Part C5272680 -> C22392391; Voltage Rating 50V -> 35V
- C144, C147, C185: footprint Capacitor_SMD:C_1206_3216Metric -> Capacitor_SMD:C_0805_2012Metric; LCSC Part C48579675 -> C98190; Voltage Rating 16V -> 10V
- C155, C157, C186: footprint Capacitor_SMD:C_1206_3216Metric -> Capacitor_SMD:C_0603_1608Metric; LCSC Part C48579675 -> C2762594
- C156: value 1uF -> 10uF; footprint Capacitor_SMD:C_0402_1005Metric -> Capacitor_SMD:C_0603_1608Metric; LCSC Part C53426846 -> C22392391; Voltage Rating 25V -> 16V
- C187: value 22uF -> 10uF; footprint Capacitor_SMD:C_1206_3216Metric -> Capacitor_SMD:C_0603_1608Metric; LCSC Part C48579675 -> C22392391
- L5: value 3.3uH 11A Sat -> 3.3uH
- R114: footprint Resistor_SMD:R_0402_1005Metric -> Resistor_SMD:R_0402_1005Metric_Pad0.72x0.64mm_HandSolder
Connections:
- net +3V3: now also C190.2, C191.2, C192.2
- net GND: now also C124.1, C128.1, C143.1, C177.2, C188.2, C189.2, C190.1, C191.1, C192.1; no longer C124.2, C128.2, C143.2
- net VSYS: now also C124.2, C128.2, C143.2, C177.1, C188.1, C189.1; no longer C124.1, C128.1, C143.1
Other:
- note added: "2 x 10uF 0603"
- note added: "3 x 10uF 0603 THANK ME LATER"
- note added: "3 x 22uF"
- note removed: "2 x 10uF 1206"
- note removed: "5 x 22uF"
- moved on the sheet: C126, R113, R119

Commit message: assign lcsc part numbers
Parts:
- R113, R119, R132: LCSC Part C2902636 -> C54951138
- R114, R120: LCSC Part C1883546 -> C54530672
- R128: LCSC Part (none) -> C100525
Changed lines of the file:
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@@
 			)
 		)
-		(property "LCSC Part" ""
+		(property "LCSC Part" "C100525"
 			(at 219.71 87.63 0)
 			(hide yes)
@@
 			)
 		)
-		(property "LCSC Part" "C2902636"
+		(property "LCSC Part" "C54951138"
 			(at 132.08 60.96 0)
 			(hide yes)
@@
 			)
 		)
-		(property "LCSC Part" "C2902636"
+		(property "LCSC Part" "C54951138"
 			(at 256.54 132.08 0)
 			(hide yes)
@@
 			)
 		)
-		(property "LCSC Part" "C2902636"
+		(property "LCSC Part" "C54951138"
 			(at 120.65 144.78 0)
 			(hide yes)
@@
 			)
 		)
-		(property "LCSC Part" "C1883546"
+		(property "LCSC Part" "C54530672"
 			(at 127 158.75 0)
 			(hide yes)
@@
 			)
 		)
-		(property "LCSC Part" "C1883546"
+		(property "LCSC Part" "C54530672"
 			(at 142.24 74.93 0)
 			(hide yes)

Commit message: new part numbers for out of stock components
Parts:
- R129: LCSC Part C861797 -> C705755
Changed lines of the file:
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@@
 			)
 		)
-		(property "LCSC Part" "C861797"
+		(property "LCSC Part" "C705755"
 			(at 231.14 66.04 0)
 			(hide yes)
@@
 			(at 231.14 66.04 0)
 			(hide yes)
+			(show_name no)
+			(do_not_autoplace no)
+			(effects
+				(font
+					(size 1.27 1.27)
+				)
+			)
+		)
+		(property "Capacitor Rating" ""
+			(at 231.14 66.04 0)
+			(hide yes)

Commit message: backup before switching to kicad-nightly
Parts:
- TP7: now left out of the parts list
Changed lines of the file:
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@@
 		(body_style 1)
 		(exclude_from_sim no)
-		(in_bom yes)
+		(in_bom no)
 		(on_board yes)
 		(in_pos_files yes)

Commit message: lots of fixes!
Parts:
- C144, C147, C185: LCSC Part C98190 -> C602037
- C155, C157, C186: LCSC Part C2762594 -> C22367828
- L4: LCSC Part C48391620 -> C439019
Other:
- moved on the sheet: L4
Changed lines of the file:
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@@
 (kicad_sch
-	(version 20260306)
+	(version 20260830)
 	(generator "eeschema")
-	(generator_version "10.0")
+	(generator_version "10.99")
 	(paper "A4")
 	(title_block
@@
 			(font
 				(size 2.794 2.794)
-				(thickness 0.5588)
+				(thickness 0.3493)
 				(bold yes)
 			)
@@
 			(font
 				(size 2.794 2.794)
-				(thickness 0.5588)
+				(thickness 0.3493)
 				(bold yes)
 			)
@@
 	(wire
 		(pts
+			(xy 125.73 161.29) (xy 127 161.29)
+		)
+		(stroke
+			(width 0)
+			(type default)
+		)
+	)
+	(wire
+		(pts
 			(xy 132.08 68.58) (xy 127 68.58)
 		)
@@
 	(wire
 		(pts
-			(xy 116.84 161.29) (xy 119.38 161.29)
+			(xy 116.84 161.29) (xy 118.11 161.29)
 		)
 		(stroke
@@
 			)
 		)
-		(property "LCSC Part" "C98190"
+		(property "LCSC Part" "C602037"
 			(at 135.89 163.83 0)
 			(hide yes)
@@
 			)
 		)
+		(property "MPN" ""
+			(at 135.89 163.83 0)
+			(hide yes)
+			(show_name no)
+			(do_not_autoplace no)
+			(effects
+				(font
+					(size 1.27 1.27)
+				)
+			)
+		)
 		(pin "1"
 		)
@@
 			)
 		)
-		(property "LCSC Part" "C2762594"
+		(property "LCSC Part" "C22367828"
 			(at 154.94 80.01 0)
 			(hide yes)
@@
 			)
 		)
-		(property "LCSC Part" "C98190"
+		(property "LCSC Part" "C602037"
 			(at 139.7 163.83 0)
 			(hide yes)
@@
 			)
 		)
+		(property "MPN" ""
+			(at 139.7 163.83 0)
+			(hide yes)
+			(show_name no)
+			(do_not_autoplace no)
+			(effects
+				(font
+					(size 1.27 1.27)
+				)
+			)
+		)
 		(pin "1"
 		)
@@
 			)
 		)
-		(property "LCSC Part" "C98190"
+		(property "LCSC Part" "C602037"
 			(at 132.08 163.83 0)
 			(hide yes)
@@
 			)
 		)
+		(property "MPN" ""
+			(at 132.08 163.83 0)
+			(hide yes)
+			(show_name no)
+			(do_not_autoplace no)
+			(effects
+				(font
+					(size 1.27 1.27)
+				)
+			)
+		)
 		(pin "1"
 		)
@@
 			)
 		)
-		(property "LCSC Part" "C2762594"
+		(property "LCSC Part" "C22367828"
 			(at 151.13 80.01 0)
 			(hide yes)
@@
 			)
 		)
-		(property "LCSC Part" "C2762594"
+		(property "LCSC Part" "C22367828"
 			(at 147.32 80.01 0)
 			(hide yes)
@@
 	(symbol
 		(lib_id "Device:L")
-		(at 123.19 161.29 90)
+		(at 121.92 161.29 90)
 		(unit 1)
 		(body_style 1)
@@
 		(dnp no)
 		(property "Reference" "L4"
-			(at 123.19 159.258 90)
+			(at 121.92 159.258 90)
 			(show_name no)
 			(do_not_autoplace no)
@@
 		)
 		(property "Value" "2.2uH"
-			(at 123.19 162.814 90)
+			(at 121.92 162.814 90)
 			(show_name no)
 			(do_not_autoplace no)
@@
 		)
 		(property "Footprint" "Inductor_SMD:L_Sunlord_MWSA1003S"
-			(at 123.19 161.29 0)
+			(at 121.92 161.29 0)
 			(hide yes)
 			(show_name no)
@@
 		)
 		(property "Datasheet" "https://www.lcsc.com/datasheet/C48391620.pdf?spm=wm.sxq.inf.ggs___wm.fly.bg.0.stp&lcsc_vid=FFRXA1JWFVgIUQBQQAAIUVdWQlILUlEHFFJcUFIATlgxVlNeQFdcUFJXQFZfXztW"
-			(at 123.19 161.29 0)
+			(at 121.92 161.29 0)
 			(hide yes)
 			(show_name no)
@@
 		)
 		(property "Description" "Inductor"
-			(at 123.19 161.29 0)
+			(at 121.92 161.29 0)
 			(hide yes)
 			(show_name no)
@@
 			)
 		)
-		(property "LCSC Part" "C48391620"
-			(at 123.19 161.29 0)
+		(property "LCSC Part" "C439019"
+			(at 121.92 161.29 0)
 			(hide yes)
 			(show_name no)
@@
 		)
 		(property "Voltage Rating" ""
-			(at 123.19 161.29 0)
+			(at 121.92 161.29 0)
 			(hide yes)
 			(show_name no)
@@
 		)
 		(property "Tolerance" ""
-			(at 123.19 161.29 0)
+			(at 121.92 161.29 0)
 			(hide yes)
 			(show_name no)
@@
 		)
 		(property "Capacitor Rating" ""
-			(at 123.19 161.29 0)
+			(at 121.92 161.29 0)
 			(hide yes)
 			(show_name no)

Commit message: change magnetometer capacitance
Parts:
- added C165: 22uF, Capacitor_SMD:C_0603_1608Metric, symbol Device:C_Small
- R128: value 750 -> 549; LCSC Part C100525 -> (none)
Connections:
- net +5V: now also C165.1
- net GND: now also C165.2
Other:
- note added: "402k/101k at 0.1%, 4.980V nominal"
- note added: "549 ohms is below what's recommended but idc"
- note removed: "402k/100k at 0.1%, 5.020V nominal"
