File: rails.kicad_sch (KiCad schematic)
At the start: 96 parts, among them Q15 2N7002, U13 LM61460AASQRJRRQ1, U14 LM61460AASQRJRRQ1, U15 TPS259474ARPWR, U16 SN74LVC1G74, Y2 SX1M4.000M10F30TNN

Commit message: replot schematic
Other:
- note added: "3 x 10uF 0603"
- note removed: "3 x 10uF 0603 THANK ME LATER"
- moved on the sheet: C122, C123, C124, C125, C126, C127, C128, C129, C131, C133, C135, C136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
