File: parsnip.kicad_sch (KiCad schematic)
At the start: 67 parts, among them J1 SPI BUS, J2 I2C3, J3 I2C1, J4 I2C2, J5 e-Ink Display Connector, J6 UART0, SW1 ESP_RESET, SW2 BOOT, U1 ESP32-S3-WROOM-1-N16R8, Y1 32.768kHz

Commit message: checkpoint: board/schematic state before scripted PCB fixes
Ryan's work in progress as of 2026-09-24 23:12: Q5/Q6 SMD type, fiducials,
U8 power-pin pours (P1-1), TH1/TH5 moved (P1-2, routing unfinished).
Also drops docs/pcb-fix-checklist.md (merged into the gitignored docs/TODO.md).

Co-Authored-By: Claude Opus 5.5 <noreply@anthropic.com>
Parts:
- added FID1, FID2, FID3: Fiducial, Fiducial:Fiducial_1mm_Mask2mm, symbol Mechanical:Fiducial
