File: parsnip.kicad_sch (KiCad schematic)
At the start: 70 parts, among them J1 SPI BUS, J2 I2C3, J3 I2C1, J4 I2C2, J5 e-Ink Display Connector, J6 UART0, SW1 ESP_RESET, SW2 BOOT, U1 ESP32-S3-WROOM-1-N16R8, Y1 32.768kHz

Commit message: nearly set to order!
Connections:
- net GND: now also J3.3 (Pin_3), J4.3 (Pin_3); no longer J3.2 (Pin_2), J4.2 (Pin_2)
- net I2C_HOST_SCL: now also J3.4 (Pin_4), J4.4 (Pin_4); no longer J3.3 (Pin_3), J4.3 (Pin_3)
- net I2C_HOST_SDA: now also J3.2 (Pin_2), J4.2 (Pin_2); no longer J3.4 (Pin_4), J4.4 (Pin_4)
Other:
- note added: "QWIIC Connector"
- moved on the sheet: C17, C3, C8, F2, F3, JP3, JP4, JP5, R20, R21, R22, R23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
