File: parsnip.kicad_sch (KiCad schematic)
At the start: 42 parts, among them SW1 ESP_RESET, SW2 BOOT, U1 ESP32-S3-WROOM-1-N16R8, Y1 32.768kHz

Commit message: schematic reorganization
Connections:
- net BUSY_DISPLAY renamed GPIO_5
- net CS_BUS renamed GPIO_38
- net CS_DISPLAY renamed GPIO_17
- net D/C_DISPLAY renamed GPIO_18
- net RESET_DISPLAY renamed GPIO_6
Other:
- sheet Connectors ports: added BUSY_DISPLAY, CS_BUS, CS_DISPLAY, D/C_DISPLAY, RESET_DISPLAY; removed none
- sheet Peripherals ports: added IO_P07; removed none
- moved on the sheet: C17, C6, C7, JP1, JP2, JP3, JP4, JP5, R12, R13, R18, R19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

Commit message: replot schematic
Other:
- moved on the sheet: C10, C11, C182, C5, C6, C7, R10, R11, R12, R13, R14, R15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

Commit message: minor bug
Other:
- moved on the sheet: TP15
Changed lines of the file:
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@@
 	(wire
 		(pts
-			(xy 177.8 64.77) (xy 194.31 64.77)
+			(xy 176.53 68.58) (xy 193.04 68.58)
 		)
 		(stroke
@@
 	)
 	(label "P16"
-		(at 194.31 69.85 180)
+		(at 193.04 73.66 180)
 		(effects
 			(font
@@
 	)
 	(label "P17"
-		(at 194.31 73.66 180)
+		(at 193.04 77.47 180)
 		(effects
 			(font
@@
 	)
 	(label "GPIO_46"
-		(at 194.31 60.96 180)
+		(at 193.04 64.77 180)
 		(effects
 			(font
@@
 	)
 	(label "P07"
-		(at 194.31 77.47 180)
+		(at 193.04 81.28 180)
 		(effects
 			(font
@@
 	(symbol
 		(lib_id "Connector:TestPoint_Probe")
-		(at 177.8 64.77 90)
+		(at 176.53 68.58 90)
 		(unit 1)
 		(body_style 1)
@@
 		(fields_autoplaced yes)
 		(property "Reference" "TP15"
-			(at 176.2125 57.15 90)
+			(at 174.9425 60.96 90)
 			(show_name no)
 			(do_not_autoplace no)
@@
 		)
 		(property "Value" "GPIO_EXP_RESET"
-			(at 176.2125 59.69 90)
+			(at 174.9425 63.5 90)
 			(show_name no)
 			(do_not_autoplace no)
@@
 		)
 		(property "Footprint" "TestPoint:TestPoint_Pad_D1.5mm"
-			(at 177.8 59.69 0)
+			(at 176.53 63.5 0)
 			(hide yes)
 			(show_name no)
@@
 		)
 		(property "Datasheet" ""
-			(at 177.8 59.69 0)
+			(at 176.53 63.5 0)
 			(hide yes)
 			(show_name no)
@@
 		)
 		(property "Description" "test point (alternative probe-style design)"
-			(at 177.8 64.77 0)
+			(at 176.53 68.58 0)
 			(hide yes)
 			(show_name no)
@@
 	)
 	(sheet
-		(at 194.31 57.15)
-		(size 30.48 26.67)
+		(at 193.04 60.96)
+		(size 34.29 24.13)
 		(exclude_from_sim no)
 		(in_bom yes)
@@
 		)
 		(property "Sheetname" "Peripherals"
-			(at 194.31 56.4384 0)
+			(at 193.04 60.2484 0)
 			(show_name no)
 			(do_not_autoplace no)
@@
 		)
 		(property "Sheetfile" "peripherals.kicad_sch"
-			(at 194.31 84.4046 0)
+			(at 193.04 85.6746 0)
 			(show_name no)
 			(do_not_autoplace no)
@@
 		)
 		(pin "LED_DIN" input
-			(at 194.31 60.96 180)
+			(at 193.04 64.77 180)
 			(effects
 				(font
@@
 		)
 		(pin "RESET_IOEXP" input
-			(at 194.31 64.77 180)
+			(at 193.04 68.58 180)
 			(effects
 				(font
@@
 		)
 		(pin "IO_P16" input
-			(at 194.31 69.85 180)
+			(at 193.04 73.66 180)
 			(effects
 				(font
@@
 		)
 		(pin "IO_P17" input
-			(at 194.31 73.66 180)
+			(at 193.04 77.47 180)
 			(effects
 				(font
@@
 		)
 		(pin "IO_P07" input
-			(at 194.31 77.47 180)
+			(at 193.04 81.28 180)
 			(effects
 				(font

Commit message: kicad updates
Parts:
- added FID4, FID5, FID6: Fiducial, Fiducial:Fiducial_1mm_Mask2mm, symbol Mechanical:Fiducial

Commit message: todo fixes
Parts:
- U1: value ESP32-S3-WROOM-1-N16R8 -> ESP32-S3-WROOM-1U-N16R8; LCSC Part C2913202 -> C3013946; MPN ESP32-S3-WROOM-1-N16R8 -> ESP32-S3-WROOM-1U-N16R8; Note (none) -> WROOM-1 (PCB antenna) footprint kept on purpose: same land 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
Changed lines of the file:
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@@
 			)
 		)
-		(property "Value" "ESP32-S3-WROOM-1-N16R8"
+		(property "Value" "ESP32-S3-WROOM-1U-N16R8"
 			(at 110.0933 76.2 0)
 			(show_name no)
@@
 			)
 		)
-		(property "Description" "MODULE Wi-Fi 802.11b/g/n + Bluetooth 5 LE, ESP32-S3, 16MB flash, 8MB octal PSRAM, PCB antenna"
+		(property "Description" "MODULE Wi-Fi 802.11b/g/n + Bluetooth 5 LE, ESP32-S3, 16MB flash, 8MB octal PSRAM, U.FL antenna connector"
 			(at 107.188 143.002 0)
 			(hide yes)
@@
 			)
 		)
-		(property "MPN" "ESP32-S3-WROOM-1-N16R8"
+		(property "MPN" "ESP32-S3-WROOM-1U-N16R8"
 			(at 86.614 75.184 0)
 			(hide yes)
@@
 			)
 		)
-		(property "LCSC Part" "C2913202"
+		(property "Note" "WROOM-1 (PCB antenna) footprint kept on purpose: same land pattern as the -1U (ds fig 11-1/11-2), so ESP32-S3-WROOM-1-N16R8 (C2913202) fits as-is. Its antenna keepout only matters for that variant."
+			(at 86.614 75.184 0)
+			(hide yes)
+			(show_name no)
+			(do_not_autoplace no)
+			(effects
+				(font
+					(size 1.27 1.27)
+				)
+			)
+		)
+		(property "LCSC Part" "C3013946"
 			(at 107.95 104.14 0)
 			(hide yes)
