File: lora.kicad_sch (KiCad schematic)
At the start: 30 parts, among them J13 SMA-KE-347-H13.5-1.6, Q14 2N7002, U12 E22P-915M30S

Commit message: schematic: add D24/D25 PZU12B2L zeners, Q_NMOS_SGD symbol, misc sheet edits
Co-Authored-By: Claude Opus 5.5 <noreply@anthropic.com>
Other:
- note added: "DC-shorted antenna only unless JP15 is cut Passive antenna only"
- note removed: "DC-shorted antenna only unless JP8 is cut Passive antenna only"
Changed lines of the file:
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@@
 		)
 	)
-	(text "DC-shorted antenna only unless JP8 is cut\nPassive antenna only"
+	(text "DC-shorted antenna only unless JP15 is cut\nPassive antenna only"
 		(exclude_from_sim no)
 		(at 80.518 138.938 0)

Commit message: checkpoint: schematic WIP before battery -> charger rename
Connectors and Overview sheets, LSM6DSV16X/TPS22945/charger datasheets,
and in-progress edits across all sheets, committed as-is so the rename
diff stands alone.

Co-Authored-By: Claude Opus 5.5 <noreply@anthropic.com>
Other:
- title: LoRa Module / LoRa Antenna -> LoRa (E22P-915M30S) & Antenna
Changed lines of the file:
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@@
 	(paper "A4")
 	(title_block
-		(title "LoRa Module / LoRa Antenna")
+		(title "LoRa (E22P-915M30S) & Antenna")
 		(date "2026-08-24")
 		(company "LimesKey")
