File: lora.kicad_sch (KiCad schematic)
At the start: 29 parts, among them J13 SMA-KE-347-H13.5-1.6, Q14 2N7002, U12 E22P-915M30S

Commit message: Netclasses: label the classed nets, add missing members
Netclass patterns keyed to KiCad's refdes-derived names (Net-(D18-A2) etc.)
drop out of their class silently on re-annotation. Local labels now name 14
of those nets (sheets + board renamed together; connectivity unchanged).

- RF_50OHM: LoRa LPF in/out + SMA, GNSS SMA + bias node now by label.
- RF_50OHM_MS: GNSS_UFL by label; width 0.30 -> 0.34 mm (50 ohm at 0.8 mm
  side clearance; 0.30 solves to 53 ohm).
- PWR_HIGH: + CHG_VBUS, /Charger/SW1, SW2, CHG_BAT, VAC1_MID, /BMS/CELL_BOT,
  BMS FET mid (full pack / charge current, previously Default).
- PWR_RAIL: + buck switch nodes, LORA_5V (E22P supply), SOLAR, VAC2_MID,
  LED 5V connector feed.
- USB_DIFF: + the six USB data nets; clearance 0.20 -> 0.15 mm (FS USB,
  matches the routed pairs).
- Root-hierarchy patterns written as */Sheet/NAME: the GUI names these
  /Root/Sheet/NAME, kicad-cli parity /Sheet/NAME.
- 8 nets had no spot for a label clear of existing text; they keep their
  current name plus the intended label name as a second pattern.
- .dru unfused_pack_plus rule names /BMS/CELL_TOP and /BMS/CELL_BOT.

Verified: knet diff (renames only), refilled DRC and ERC identical to
before, kpcb sync clean.

Co-Authored-By: Claude Opus 5.5 <noreply@anthropic.com>
Connections:
- net LORA_5V: now reaches C117.1, C118.1, C119.1, C120.1, D19.2 (A2), R100.2, U12.10 (VCC), U12.9 (VCC)
- net LORA_LPF_OUT: now reaches C114.1, FL2.4 (IO), JP14.1 (A), R95.2
- net LORA_LPF_IN: now reaches C115.2, FL2.8 (IO), JP14.2 (B)
- net LORA_SMA: now reaches C113.1, D18.2 (A2), J13.1 (In), L3.2, R95.1
Changed lines of the file:
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@@
+		)
+	)
+	(label "LORA_SMA"
+		(at 66.04 156.21 180)
+		(effects
+			(font
+				(size 1.27 1.27)
+			)
+			(justify right bottom)
+		)
+	)
+	(label "LORA_LPF_OUT"
+		(at 77.47 162.56 0)
+		(effects
+			(font
+				(size 1.27 1.27)
+			)
+			(justify left bottom)
+		)
+	)
+	(label "LORA_LPF_IN"
+		(at 120.65 156.21 270)
+		(effects
+			(font
+				(size 1.27 1.27)
+			)
+			(justify right bottom)
+		)
+	)
+	(label "LORA_5V"
+		(at 185.42 83.82 0)
+		(effects
+			(font
+				(size 1.27 1.27)
+			)
+			(justify left bottom)
 		)
 	)
