File: overview.kicad_sch (KiCad schematic)
At the start: 0 parts

Commit message: schematic: front matter - cover, block diagram, power tree (pages 1-3)
Structure follows the NXP i.MX8M EVK and BeaglePlay schematic sets.
- overview.kicad_sch (p1): cover with page list and revision history as
  KiCad tables (rows link to their pages) and general notes.
- block_diagram.kicad_sch (p2): ESP32-S3-centred block diagram with buses,
  control lines and I2C addresses.
- power_tree.kicad_sch (p3): inputs, charger, bucks, eFuses and loads,
  one colour per rail.
- parsnip.kicad_pro: Block Diagram and Power Tree registered as top-level
  sheets 2-3; REV/DATE text variables (1.1, 2026-10-03) for the new title
  blocks.
- Pages 2-10 renumbered to 4-12 (page lines only).

Every refdes, value and I2C address on p2/p3 was checked against the
merged netlist or datasheets on 2026-10-03. New sheets were re-saved with
kicad-cli sch upgrade so the first GUI save doesn't reformat them.

Verified: netlist unchanged (462 comps / 295 nets, now 12 sheets), ERC
unchanged (330, no findings on the new sheets), PDF prints Id 1/12..12/12
in order, kpcb sync unchanged.

Co-Authored-By: Claude Opus 5.5 <noreply@anthropic.com>
Other:
- note added: "1."
- note added: "2."
- note added: "3."
- note added: "4."
- note added: "5."
- note added: "6."
- note added: "7."
- note added: "An overbar on a pin or net name denotes an active-low signal."
- note added: "DNP = do not populate. DNP symbols are drawn with a red X."
- note added: "Labels with the same name are connected. Top-level sheets join through global labels and power symbols, subsheets of Root through sheet pins."
- note added: "Meshtastic LoRa mesh node, 915 MHz"
- note added: "NOTES, UNLESS OTHERWISE SPECIFIED:"
- note added: "PAGE LIST"
- note added: "PARSNIP-NODE"
- note added: "PWR_FLAG symbols are for ERC only and are not parts."
- note added: "REVISION HISTORY"
- note added: "Resistance in ohms, capacitance in farads. All voltages are DC."
- note added: "Resistors and capacitors are 0402."
- note added: "Schematic"
- note added: "Some symbols are edited in the schematic. Do not run Tools > Update Symbols from Library."
- title: Block Diagram & Notes -> Cover
