File: usb_interface.kicad_sch (KiCad schematic)
At the start: 57 parts, among them J7 USB4105-GF-A-060, J8 PD_I2C DEBUG, Q1 CSD23280F3, Q2 CSD15380F3, Q3 CSD23280F3, Q4 CSD15380F3, U21 M24512-DFMC6TG, U3 TVS2200DRV, U4 TPD8S300A, U5 TPS25751DREFR

Commit message: checkpoint: schematic WIP before battery -> charger rename
Connectors and Overview sheets, LSM6DSV16X/TPS22945/charger datasheets,
and in-progress edits across all sheets, committed as-is so the rename
diff stands alone.

Co-Authored-By: Claude Opus 5.5 <noreply@anthropic.com>
Other:
- note removed: "7 x 10uF"
- title: USB Interface -> USB-C Port: PD, OVP/ESD, Data
- moved on the sheet: C20, C25, Q1, Q2, Q3, Q4, R28, R29, R30, R31
