File: charger.kicad_sch (KiCad schematic)
At the start: 61 parts, among them J10 SOLAR, Q10 SI2308, Q11 CSD17577Q3A, Q7 CSD18512Q5B, Q8 CSD18512Q5B, Q9 SI2308, SW3 RESET, U8 BQ25798

Commit message: replot schematic
Parts:
- SW3: now in the parts list
Changed lines of the file:
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@@
 		(body_style 1)
 		(exclude_from_sim no)
-		(in_bom no)
+		(in_bom yes)
 		(on_board yes)
 		(in_pos_files yes)

Commit message: minor bug
Changed lines of the file:
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@@
 	(text "${TITLE}"
 		(exclude_from_sim no)
-		(at 274.828 -17.526 0)
+		(at 238.76 46.482 0)
 		(effects
 			(font
@@
 			)
 		)
-		(property "Description" "RES 30.1kΩ ±0.1% 25ppm 100mW 0603 thin film"
+		(property "Description" "RES 32.4kΩ ±0.1% 100mW 0603"
 			(at 186.69 151.13 0)
 			(hide yes)
