File: charger.kicad_sch (KiCad schematic)
At the start: 61 parts, among them J10 SOLAR, Q10 SI2308, Q11 CSD17577Q3A, Q7 CSD18512Q5B, Q8 CSD18512Q5B, Q9 SI2308, SW3 RESET, U8 BQ25798

Commit message: Netclasses: label the classed nets, add missing members
Netclass patterns keyed to KiCad's refdes-derived names (Net-(D18-A2) etc.)
drop out of their class silently on re-annotation. Local labels now name 14
of those nets (sheets + board renamed together; connectivity unchanged).

- RF_50OHM: LoRa LPF in/out + SMA, GNSS SMA + bias node now by label.
- RF_50OHM_MS: GNSS_UFL by label; width 0.30 -> 0.34 mm (50 ohm at 0.8 mm
  side clearance; 0.30 solves to 53 ohm).
- PWR_HIGH: + CHG_VBUS, /Charger/SW1, SW2, CHG_BAT, VAC1_MID, /BMS/CELL_BOT,
  BMS FET mid (full pack / charge current, previously Default).
- PWR_RAIL: + buck switch nodes, LORA_5V (E22P supply), SOLAR, VAC2_MID,
  LED 5V connector feed.
- USB_DIFF: + the six USB data nets; clearance 0.20 -> 0.15 mm (FS USB,
  matches the routed pairs).
- Root-hierarchy patterns written as */Sheet/NAME: the GUI names these
  /Root/Sheet/NAME, kicad-cli parity /Sheet/NAME.
- 8 nets had no spot for a label clear of existing text; they keep their
  current name plus the intended label name as a second pattern.
- .dru unfused_pack_plus rule names /BMS/CELL_TOP and /BMS/CELL_BOT.

Verified: knet diff (renames only), refilled DRC and ERC identical to
before, kpcb sync clean.

Co-Authored-By: Claude Opus 5.5 <noreply@anthropic.com>
Connections:
- net CHG_BAT: now reaches C84.2, C85.2, Q11.1 (S), Q11.2 (S), Q11.3 (S), U8.22 (BAT), U8.23 (BAT)
- net VAC2_MID: now reaches D25.2 (A), Q10.2 (S), Q9.2 (S)
- net VAC1_MID: now reaches D24.2 (A), Q7.1 (S), Q8.1 (S)
- net SW1: now reaches C75.2, L1.1, R65.1, U8.28 (SW1)
- net SW2: now reaches C76.1, L1.2, R64.1, U8.26 (SW2)
Changed lines of the file:
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@@
+		)
+	)
+	(label "VAC2_MID"
+		(at 104.14 68.58 180)
+		(effects
+			(font
+				(size 1.27 1.27)
+			)
+			(justify right bottom)
+		)
+	)
+	(label "VAC1_MID"
+		(at 102.87 29.21 180)
+		(effects
+			(font
+				(size 1.27 1.27)
+			)
+			(justify right bottom)
+		)
+	)
+	(label "SW2"
+		(at 204.47 86.36 0)
+		(effects
+			(font
+				(size 1.27 1.27)
+			)
+			(justify left bottom)
+		)
+	)
+	(label "SW1"
+		(at 204.47 74.93 0)
+		(effects
+			(font
+				(size 1.27 1.27)
+			)
+			(justify left bottom)
+		)
+	)
+	(label "CHG_BAT"
+		(at 208.28 114.3 0)
+		(effects
+			(font
+				(size 1.27 1.27)
+			)
+			(justify left bottom)
 		)
 	)
