File: charger.kicad_sch (KiCad schematic)
At the start: 61 parts, among them J10 SOLAR, Q10 SI2308, Q11 CSD17577Q3A, Q7 CSD18512Q5B, Q8 CSD18512Q5B, Q9 SI2308, SW3 RESET, U8 BQ25798

Commit message: symbol property changes -- chores
Parts:
- C81, C83, R64, R65: now in the parts list
Changed lines of the file:
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@@
 		(in_bom no)
 		(on_board yes)
-		(in_pos_files yes)
+		(in_pos_files no)
 		(dnp no)
 		(property "Reference" "TP4"
@@
 		(body_style 1)
 		(exclude_from_sim no)
-		(in_bom no)
+		(in_bom yes)
 		(on_board yes)
 		(in_pos_files yes)
@@
 		(body_style 1)
 		(exclude_from_sim no)
-		(in_bom no)
+		(in_bom yes)
 		(on_board yes)
 		(in_pos_files yes)
@@
 		(body_style 1)
 		(exclude_from_sim no)
-		(in_bom no)
+		(in_bom yes)
 		(on_board yes)
 		(in_pos_files yes)
@@
 		(body_style 1)
 		(exclude_from_sim no)
-		(in_bom no)
+		(in_bom yes)
 		(on_board yes)
 		(in_pos_files yes)

Commit message: routing + part number changes
Parts:
- L1: Manufacturer Sunlord -> TAI-TECH
Changed lines of the file:
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@@
 			)
 		)
-		(property "Manufacturer" "Sunlord"
+		(property "Manufacturer" "TAI-TECH"
 			(at 200.66 81.28 0)
 			(hide yes)
