File: gnss.kicad_sch (KiCad schematic)
At the start: 71 parts, among them J11 SMA-KE-347-H13.5-1.6, J12 U.FL, SW4 RESET_GNSS, SW5 SAFEBOOT_GNSS, U10 TPS7A2033PDBVR, U11 TPS259474LRPWR, U6 TPS22945DCKR, U9 NEO-F10N

Commit message: schematic reorganization
Parts:
- added R136: 100k, Resistor_SMD:R_0402_1005Metric, symbol Device:R_Small
Connections:
- net 3V3_GNSS: now also R136.2
- net ANT_FAULT: now also R136.1
Other:
- moved on the sheet: C101, D12, D16, FB1, JP10, JP11, JP12, R67, R68, R70, R71, R72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

Commit message: replot schematic
Parts:
- BT3: now fitted
Changed lines of the file:
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@@
 		(in_bom yes)
 		(on_board yes)
-		(in_pos_files yes)
-		(dnp yes)
+		(in_pos_files no)
+		(dnp no)
 		(property "Reference" "BT3"
 			(at 142.748 25.4 90)

Commit message: minor bug
Parts:
- BT3: now left out of the parts list
- R74: LCSC Part (none) -> C510088; MPN (none) -> ESR03EZPF10R0; Manufacturer (none) -> ROHM
Changed lines of the file:
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@@
 		(body_style 1)
 		(exclude_from_sim no)
-		(in_bom yes)
+		(in_bom no)
 		(on_board yes)
 		(in_pos_files no)
@@
 			)
 		)
-		(property "Datasheet" ""
+		(property "Datasheet" "https://www.lcsc.com/datasheet/C510088.pdf"
 			(at 44.45 171.45 0)
 			(hide yes)
@@
 			)
 		)
-		(property "Description" ""
+		(property "Description" "RES 10Ω ±1% 250mW 0603"
 			(at 44.45 171.45 0)
 			(hide yes)
@@
 			)
 		)
-		(property "MPN" ""
+		(property "MPN" "ESR03EZPF10R0"
 			(at 44.45 173.228 90)
 			(hide yes)
@@
 			)
 		)
-		(property "Manufacturer" ""
+		(property "Manufacturer" "ROHM"
 			(at 44.45 173.228 90)
 			(hide yes)
@@
 			)
 		)
-		(property "LCSC Part" ""
+		(property "LCSC Part" "C510088"
 			(at 44.45 171.45 0)
 			(hide yes)
