File: bms.kicad_sch (KiCad schematic)
At the start: 50 parts, among them J9 BAT_PORT, Q16 TPN2R203NC, Q5 AON7544, Q6 AON7544, U7 MAX17320G22+

Commit message: Netclasses: label the classed nets, add missing members
Netclass patterns keyed to KiCad's refdes-derived names (Net-(D18-A2) etc.)
drop out of their class silently on re-annotation. Local labels now name 14
of those nets (sheets + board renamed together; connectivity unchanged).

- RF_50OHM: LoRa LPF in/out + SMA, GNSS SMA + bias node now by label.
- RF_50OHM_MS: GNSS_UFL by label; width 0.30 -> 0.34 mm (50 ohm at 0.8 mm
  side clearance; 0.30 solves to 53 ohm).
- PWR_HIGH: + CHG_VBUS, /Charger/SW1, SW2, CHG_BAT, VAC1_MID, /BMS/CELL_BOT,
  BMS FET mid (full pack / charge current, previously Default).
- PWR_RAIL: + buck switch nodes, LORA_5V (E22P supply), SOLAR, VAC2_MID,
  LED 5V connector feed.
- USB_DIFF: + the six USB data nets; clearance 0.20 -> 0.15 mm (FS USB,
  matches the routed pairs).
- Root-hierarchy patterns written as */Sheet/NAME: the GUI names these
  /Root/Sheet/NAME, kicad-cli parity /Sheet/NAME.
- 8 nets had no spot for a label clear of existing text; they keep their
  current name plus the intended label name as a second pattern.
- .dru unfused_pack_plus rule names /BMS/CELL_TOP and /BMS/CELL_BOT.

Verified: knet diff (renames only), refilled DRC and ERC identical to
before, kpcb sync clean.

Co-Authored-By: Claude Opus 5.5 <noreply@anthropic.com>
Connections:
- net CELL_TOP: now reaches BT1.1 (+), F5.1, J9.2 (Pin_2), R135.2, R40.1, R42.1
- net CELL_BOT: now reaches BT2.2 (-), J9.1 (Pin_1), Q16.5 (D), Q16.6 (D), Q16.7 (D), Q16.8 (D), Q16.9 (D)
Changed lines of the file:
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@@
+		)
+	)
+	(label "CELL_BOT"
+		(at 66.04 110.49 180)
+		(effects
+			(font
+				(size 1.27 1.27)
+			)
+			(justify right bottom)
+		)
+	)
+	(label "CELL_TOP"
+		(at 71.12 67.31 0)
+		(effects
+			(font
+				(size 1.27 1.27)
+			)
+			(justify left bottom)
 		)
 	)
