File: parsnip.kicad_pcb (KiCad board)
At the start: 4 copper layers, 60 x 130 mm, 481 parts, among them J1 SPI0, J10 SOLAR, J11 SMA-KE-347-H13.5-1.6, J12 U.FL, J13 SMA-KE-347-H13.5-1.6, J14 GPIO_Expander, J15 LED 5V, J16 I2C3, J2 I2C4, J3 I2C1, J4 I2C2, J5 SPI1, J6 UART0, J7 USB4105-GF-A-060, J8 PD_I2C DEBUG, J9 BAT_PORT, Q1 CSD23280F3, Q10 SI2308, Q11 CSD17577Q3A, Q14 2N7002, Q15 2N7002, Q16 TPN2R203NC, Q2 CSD15380F3, Q3 CSD23280F3, Q4 CSD15380F3, Q5 AON7544, Q6 AON7544, Q7 CSD18512Q5B, Q8 CSD18512Q5B, Q9 SI2308, SW1 ESP_RESET, SW2 BOOT, SW3 RESET, SW4 RESET_GNSS, SW5 SAFEBOOT_GNSS, U1 ESP32-S3-WROOM-1U-N16R8, U10 TPS7A2033PDBVR, U11 TPS259474LRPWR, U12 E22P-915M30S, U13 LM61460AASQRJRRQ1, U14 LM61460AASQRJRRQ1, U15 TPS259474ARPWR, U16 SN74LVC1G74, U17 TCAL9539RTWRQ1, U18 WS2816B, U19 SN74LV1T34DCK, U2 QMC6309, U20 WS2816B, U21 M24512-DFMC6TG, U22 LSM6DSV16X, U23 TPS22945DCKR, U24 TPD2E2U06QDCKRQ1, U3 TVS2200DRV, U4 TPD8S300A, U5 TPS25751DREFR, U6 TPS22945DCKR, U7 MAX17320G22+, U8 BQ25798, U9 NEO-F10N, Y1 32.768kHz, Y2 SX1M4.000M10F30TNN

Commit message: checkpoint: board as on disk 2026-10-28 19:50 (pre-edit, includes the earlier R20 move, not yet refilled)
Co-Authored-By: Claude Opus 5.5 <noreply@anthropic.com>
Routing:
- net I2C_HOST_IRQ: track 78.5 -> 79.6 mm
- net /USB Interface/CC2: track 10.7 -> 11.2 mm
Changed lines of the file:
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@@
 		(layer "B.Cu")
 		(transform
-			(translate 126.75 150.6)
+			(translate 127.85 150.6)
 			(rotate -90)
 			(scale 1 1)
@@
 	)
 	(segment
-		(start 127.2875 151.1975)
-		(end 126.75 151.1975)
-		(width 0.5)
-		(layer "B.Cu")
-		(net "Net-(JP3-A)")
-	)
-	(segment
 		(start 125.75 139.542893)
 		(end 125.75 146.15)
@@
 		(net "Net-(D4-K)")
 	)
+	(segment
+		(start 126.75 150.0025)
+		(end 127.85 150.0025)
+		(width 0.5)
+		(layer "B.Cu")
+		(net "I2C_HOST_IRQ")
+	)
+	(segment
+		(start 127.2875 151.1975)
+		(end 127.85 151.1975)
+		(width 0.5)
+		(layer "B.Cu")
+		(net "Net-(JP3-A)")
+	)
+	(segment
+		(start 138.2 146.130947)
+		(end 138.2 146.7)
+		(width 0.2)
+		(layer "F.Cu")
+		(net "/USB Interface/CC2")
+	)
 	(zone
 		(net "/USB Interface/GPIO2")
@@
 			)
 		)
-	)
-	(zone
-		(net "Net-(JP3-A)")
-		(layer "B.Cu")
-		(hatch none 0.1)
-		(priority 30142)
-		(attr
-			(teardrop
-				(type padvia)
-			)
-		)
-		(connect_pads yes
-			(clearance 0)
-		)
-		(min_thickness 0.0254)
-		(fill yes
-			(island_removal_mode 1)
-		)
-		(polygon
-			(pts
-				(xy 127.2875 150.9475) (xy 127.254085 150.94841) (xy 127.142164 150.942795) (xy 127.078088 150.921398)
-				(xy 127.009124 150.8775) (xy 126.749 151.1975) (xy 127.009124 151.5175) (xy 127.057721 151.484162)
-				(xy 127.103998 151.462884) (xy 127.197802 151.445826) (xy 127.254085 151.44659) (xy 127.2875 151.4475)
-			)
-		)
