File: block_diagram.kicad_sch (KiCad schematic)
At the start: 0 parts

Commit message: todo fixes
Other:
- note added: "ESP32-S3-WROOM-1U"
- note removed: "ESP32-S3-WROOM-1"
Changed lines of the file:
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@@
 		)
 	)
-	(text "ESP32-S3-WROOM-1"
+	(text "ESP32-S3-WROOM-1U"
 		(exclude_from_sim no)
 		(at 144 86 0)
