File: connectors.kicad_sch (KiCad schematic)
At the start: 35 parts, among them J1 SPI BUS, J16 I2C3, J2 I2C4, J3 I2C1, J4 I2C2, J5 e-Ink Display Connector, J6 UART0, U23 TPS22945DCKR

Commit message: schematic reorganization
Parts:
- removed F3, F8: 1A hold, Fuse:Fuse_0805_2012Metric, symbol Device:Polyfuse_Small
- added C142: 1uF, Capacitor_SMD:C_0402_1005Metric, symbol Device:C_Small
- added C4: 2.2uF, Capacitor_SMD:C_0402_1005Metric, symbol Device:C_Small
- added D26, D28, D29: ESDS314DBVR, Package_TO_SOT_SMD:SOT-23-5, symbol easyeda2kicad:ESDS314DBVR-TP
- added D27: 1N5819WS, Diode_SMD:D_SOD-323, symbol Device:D_Schottky_Small
- added R23, R60: 33, Resistor_SMD:R_0402_1005Metric_Pad0.72x0.64mm_HandSolder, symbol Device:R_Small
- J1: value SPI BUS -> SPI0
- J5: value e-Ink Display Connector -> SPI1
Connections:
- net +3V3: now also D27.2 (A); no longer C8.1, C9.1
- net BUSY_DISPLAY: no longer D3.3 (I/O2)
- net CS_BUS: no longer D1.5 (I/O4)
- net CS_DISPLAY: no longer D2.4 (I/O3)
- net D/C_DISPLAY: no longer D3.1 (I/O1)
- net GND: now also U23.2 (GND), C142.2, C4.2, D26.2 (GND), D28.2 (GND), D29.2 (GND)
- net I2C_HOST_SCL: now also D26.1 (I/O1), D26.5 (I/O4), D28.1 (I/O1), D28.5 (I/O4), D29.1 (I/O1), D29.5 (I/O4), R60.1; no longer J2.4 (Pin_4)
- net I2C_HOST_SDA: now also D26.3 (I/O2), D26.4 (I/O3), D28.3 (I/O2), D28.4 (I/O3), D29.3 (I/O2), D29.4 (I/O3), R23.1; no longer J2.3 (Pin_3)
- net MISO: no longer D1.4 (I/O3)
- net MOSI: no longer D1.3 (I/O2)
- net RESET_DISPLAY: no longer D2.5 (I/O4)
- net SCK: no longer D1.1 (I/O1)
- net UART0_RX: no longer D3.5 (I/O4)
- net UART0_TX: no longer D3.4 (I/O3)
- net UART0_RX_RAW: now reaches R16.2
- net UART0_RX_RAW: now also D3.3 (I/O2), D3.4 (I/O3), J6.3 (Pin_3); no longer J6.2 (Pin_2)
- net UART0_TX_RAW: now reaches R17.2
- net UART0_TX_RAW: now also D3.1 (I/O1), D3.5 (I/O4), J6.2 (Pin_2); no longer J6.3 (Pin_3)
- net MISO_RAW: now reaches J1.5 (Pin_5), R3.2
- net MISO_RAW: now also D1.4 (I/O3)
- net CS_BUS_RAW: now reaches J1.6 (Pin_6), R4.2
- net CS_BUS_RAW: now also D1.5 (I/O4)
- net MOSI_RAW: now reaches J1.4 (Pin_4), R2.2
- net MOSI_RAW: now also D1.3 (I/O2)
- net +3V3_EXT: now reaches J16.1 (Pin_1)
- net +3V3_EXT: now also C8.1, C9.1, J4.1 (Pin_1), U23.1 (VOUT), C142.1
- net SCK_RAW: now reaches J1.3 (Pin_3), R1.2
- net SCK_RAW: now also D1.1 (I/O1)
- net at U23.4 (ON): now also U23.5 (VIN), C4.1, D27.1 (K)
- new net: J2.4 (Pin_4), R60.2
- new net: J2.3 (Pin_3), R23.2
- no-connect marks 0 -> 3
Other:
- note added: "Air Quality Sensor"
- note added: "I2C1"
- note added: "I2C2 & I2C3"
- note added: "Low-input-voltage Current-limited Load Switches With Shut Off And Auto- Restart Feature"
- note added: "QWIIC I2C4"
- note added: "SPI0"
- note added: "UART0"
- note added: "ePaper Display SPI1"
- note removed: "Air Sensor"
- moved on the sheet: C1, C13, C14, C2, C3, C8, C9, D1, D2, D3, D4, F1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

Commit message: replot schematic
Parts:
- J16, J4: now in the parts list
Changed lines of the file:
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@@
 	(title_block
 		(title "Expansion & Display Connectors")
+		(date "2026-10-05")
 		(company "LimesKey")
 	)
@@
 		(body_style 1)
 		(exclude_from_sim no)
-		(in_bom no)
+		(in_bom yes)
 		(on_board yes)
-		(in_pos_files yes)
+		(in_pos_files no)
 		(dnp no)
 		(fields_autoplaced yes)
@@
 			)
 		)
+		(property "MPN" ""
+			(at 143.51 115.57 0)
+			(hide yes)
+			(show_name no)
+			(do_not_autoplace no)
+			(effects
+				(font
+					(size 1.27 1.27)
+				)
+			)
+		)
+		(property "Manufacturer" ""
+			(at 143.51 115.57 0)
+			(hide yes)
+			(show_name no)
+			(do_not_autoplace no)
+			(effects
+				(font
+					(size 1.27 1.27)
+				)
+			)
+		)
+		(property "LCSC Part" ""
+			(at 143.51 115.57 0)
+			(hide yes)
+			(show_name no)
+			(do_not_autoplace no)
+			(effects
+				(font
+					(size 1.27 1.27)
+				)
+			)
+		)
+		(property "Voltage Rating" ""
+			(at 143.51 115.57 0)
+			(hide yes)
+			(show_name no)
+			(do_not_autoplace no)
+			(effects
+				(font
+					(size 1.27 1.27)
+				)
+			)
+		)
+		(property "Tolerance" ""
+			(at 143.51 115.57 0)
+			(hide yes)
+			(show_name no)
+			(do_not_autoplace no)
+			(effects
+				(font
+					(size 1.27 1.27)
+				)
+			)
+		)
 		(pin "2"
 		)
@@
 		(body_style 1)
 		(exclude_from_sim no)
-		(in_bom no)
+		(in_bom yes)
 		(on_board yes)
-		(in_pos_files yes)
+		(in_pos_files no)
 		(dnp no)
 		(fields_autoplaced yes)
@@
 			(at 143.51 85.09 0)
 			(hide yes)
+			(show_name no)
+			(do_not_autoplace no)
+			(effects
+				(font
+					(size 1.27 1.27)
+				)
+			)
+		)
+		(property "MPN" ""
+			(at 143.51 85.09 0)
+			(hide yes)
+			(show_name no)
+			(do_not_autoplace no)
+			(effects
+				(font
+					(size 1.27 1.27)
+				)
+			)
+		)
+		(property "Manufacturer" ""
+			(at 143.51 85.09 0)
+			(hide yes)
+			(show_name no)
+			(do_not_autoplace no)
+			(effects
+				(font
+					(size 1.27 1.27)
+				)
+			)
+		)
+		(property "LCSC Part" ""
+			(at 143.51 85.09 0)
+			(hide yes)
+			(show_name no)
+			(do_not_autoplace no)
+			(effects
+				(font
+					(size 1.27 1.27)
+				)
+			)
+		)
+		(property "Voltage Rating" ""
+			(at 143.51 85.09 0)
+			(hide yes)
+			(show_name no)
+			(do_not_autoplace no)
+			(effects
+				(font
+					(size 1.27 1.27)
+				)
+			)
+		)
+		(property "Tolerance" ""
+			(at 143.51 85.09 0)
+			(hide yes)

Commit message: minor bug
Connections:
- net I2C_HOST_SCL: no longer D26.1 (I/O1), D26.5 (I/O4)
- net I2C_HOST_SDA: no longer D26.3 (I/O2), D26.4 (I/O3)
- net UART0_RX_RAW: now also R17.2; no longer R16.2
- net UART0_TX_RAW: now also R16.2; no longer R17.2
- net I2C_HOST_SCL_RAW: now reaches J2.4 (Pin_4), R60.2
- net I2C_HOST_SCL_RAW: now also D26.1 (I/O1), D26.5 (I/O4)
- net I2C_HOST_SDA_RAW: now reaches J2.3 (Pin_3), R23.2
- net I2C_HOST_SDA_RAW: now also D26.3 (I/O2), D26.4 (I/O3)
Other:
- moved on the sheet: D26

Commit message: new prod
Parts:
- J16, J4: LCSC Part (none) -> C7509546; MPN (none) -> DS1023-1x4SF11; Manufacturer (none) -> CONNFLY Elec
Changed lines of the file:
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@@
 			)
 		)
-		(property "Datasheet" ""
+		(property "Datasheet" "https://datasheet.lcsc.com/datasheet/pdf/e746529444b0a48d4f291628523ddcfb.pdf?productCode=C7509546"
 			(at 143.51 115.57 0)
 			(hide yes)
@@
 			)
 		)
-		(property "Description" "CONN RCPT female 1x4 2.54mm, vertical THT (not in BOM)"
+		(property "Description" "CONN RCPT female 1x4 2.54mm, vertical THT"
 			(at 143.51 115.57 0)
 			(hide yes)
@@
 			)
 		)
-		(property "MPN" ""
+		(property "MPN" "DS1023-1x4SF11"
 			(at 143.51 115.57 0)
 			(hide yes)
@@
 			)
 		)
-		(property "Manufacturer" ""
+		(property "Manufacturer" "CONNFLY Elec"
 			(at 143.51 115.57 0)
 			(hide yes)
@@
 			)
 		)
-		(property "LCSC Part" ""
+		(property "LCSC Part" "C7509546"
 			(at 143.51 115.57 0)
 			(hide yes)
@@
 			)
 		)
-		(property "Datasheet" ""
+		(property "Datasheet" "https://datasheet.lcsc.com/datasheet/pdf/e746529444b0a48d4f291628523ddcfb.pdf?productCode=C7509546"
 			(at 143.51 85.09 0)
 			(hide yes)
@@
 			)
 		)
-		(property "Description" "CONN RCPT female 1x4 2.54mm, vertical THT (not in BOM)"
+		(property "Description" "CONN RCPT female 1x4 2.54mm, vertical THT"
 			(at 143.51 85.09 0)
 			(hide yes)
@@
 			)
 		)
-		(property "MPN" ""
+		(property "MPN" "DS1023-1x4SF11"
 			(at 143.51 85.09 0)
 			(hide yes)
@@
 			)
 		)
-		(property "Manufacturer" ""
+		(property "Manufacturer" "CONNFLY Elec"
 			(at 143.51 85.09 0)
 			(hide yes)
@@
 			)
 		)
-		(property "LCSC Part" ""
+		(property "LCSC Part" "C7509546"
 			(at 143.51 85.09 0)
 			(hide yes)

Commit message: routing + part number changes
Parts:
- F2: LCSC Part C6851467 -> C70158; MPN SL0805200-12V -> SL0805200
Changed lines of the file:
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@@
 			)
 		)
-		(property "Datasheet" "https://datasheet.lcsc.com/datasheet/pdf/e6a378b8a37019759bb545a349a60ab8.pdf?productCode=C6851467"
+		(property "Datasheet" "https://datasheet.lcsc.com/datasheet/pdf/e6a378b8a37019759bb545a349a60ab8.pdf?productCode=C70158"
 			(at 45.72 124.46 0)
 			(hide yes)
@@
 			)
 		)
-		(property "Description" "FUSE PTC resettable 2A hold, 4A trip, 12V, 0805"
+		(property "Description" "FUSE PTC resettable 2A hold, 4A trip, 6V, 0805"
 			(at 45.72 124.46 0)
 			(hide yes)
@@
 			)
 		)
-		(property "MPN" "SL0805200-12V"
+		(property "MPN" "SL0805200"
 			(at 40.64 125.73 0)
 			(hide yes)
@@
 			)
 		)
-		(property "LCSC Part" "C6851467"
+		(property "LCSC Part" "C70158"
 			(at 45.72 124.46 0)
 			(hide yes)
