File: power_tree.kicad_sch (KiCad schematic)
At the start: 0 parts

Commit message: todo fixes
Other:
- note added: "ESP32-S3-WROOM-1U (U1)"
- note removed: "ESP32-S3-WROOM-1 (U1)"
Changed lines of the file:
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@@
 		)
 	)
-	(text "ESP32-S3-WROOM-1 (U1)"
+	(text "ESP32-S3-WROOM-1U (U1)"
 		(exclude_from_sim no)
 		(at 257.5 105.375 0)

Commit message: symbol property changes -- chores
Other:
- note added: "J1-J3 (F1, F7, F2), J4/J16 (U23)"
- note removed: "J1-J4, J16 (F1-F3, F7, F8)"
Changed lines of the file:
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@@
 		)
 	)
-	(text "J1-J4, J16 (F1-F3, F7, F8)"
+	(text "J1-J3 (F1, F7, F2), J4/J16 (U23)"
 		(exclude_from_sim no)
 		(at 257.5 149.375 0)
